File: amepl_led.kicad_pcb (KiCad board)
At the start: 2 copper layers, 140 x 140 mm, 129 parts, among them J1 Conn_01x03_Male

Commit message: Review Korrekturen und Erstellung der Gerber Dateien
Routing:
- net GND: track 0.57 -> 0.00 mm
Other:
- board text added: "v1.0"

Commit message: Fertigstellung von v1.0
Parts:
- added J2: Conn_01x03_Male, Connector_JST:JST_XH_B3B-XH-A_1x03_P2.50mm_Vertical, B.Cu at (90.5, 156.0)
- added J3: Conn_01x04_Male, Connector_PinHeader_2.54mm:PinHeader_1x04_P2.54mm_Vertical, B.Cu at (103.0, 170.5)
- moved J1 6.00 mm to (90.5, 144.0)
Connections:
- net Net-(D1-Pad4) renamed DIN
- D64 pad 2: Net-(D64-Pad2) -> DOUT
Routing:
- net DOUT: track 0.00 -> 92.7 mm
- net DIN: track 58.6 -> 90.5 mm
Other:
- board text added: "DOUT"
