File: amepl_led.sch (KiCad schematic (older format))
At the start: 129 parts, among them J1 Conn_01x03_Male

Commit message: Fertigstellung von v1.0
Parts:
- added J2: Conn_01x03_Male, Connector_JST:JST_XH_B3B-XH-A_1x03_P2.50mm_Vertical, symbol Connector:Conn_01x03_Male
- added J3: Conn_01x04_Male, Connector_PinHeader_2.54mm:PinHeader_1x04_P2.54mm_Vertical, symbol Connector:Conn_01x04_Male
Connections:
- net +5V: now also J2.1 (Pin_1), J3.1 (Pin_1)
- net GND: now also J2.3 (Pin_3), J3.2 (Pin_2)
- net DIN: now reaches D1.4 (DIN), J1.2 (Pin_2)
- net DIN: now also J3.3 (Pin_3)
- net DOUT: now reaches D64.2 (DOUT)
- net DOUT: now also J2.2 (Pin_2), J3.4 (Pin_4)
- no-connect marks 1 -> 0
Other:
- moved on the sheet: J1
Changed lines of the file:
@@
 	6150 7150 6150 7100
 Wire Wire Line
-	6450 6800 6550 6800
-Wire Wire Line
 	10900 1350 10900 2050
 Wire Wire Line
@@
 Wire Wire Line
 	10700 5500 11050 5500
-NoConn ~ 6550 6800
 $Comp
 L Connector:Conn_01x03_Male J1
 U 1 1 618FD6DF
-P 600 1350
-F 0 "J1" H 650 1150 50  0000 C CNN
-F 1 "Conn_01x03_Male" V 550 1400 50  0000 C CNN
-F 2 "Connector_JST:JST_XH_B3B-XH-A_1x03_P2.50mm_Vertical" H 600 1350 50  0001 C CNN
-F 3 "~" H 600 1350 50  0001 C CNN
-	1    600  1350
+P 550 1350
+F 0 "J1" H 600 1150 50  0000 C CNN
+F 1 "Conn_01x03_Male" V 500 1400 50  0000 C CNN
+F 2 "Connector_JST:JST_XH_B3B-XH-A_1x03_P2.50mm_Vertical" H 550 1350 50  0001 C CNN
+F 3 "~" H 550 1350 50  0001 C CNN
+	1    550  1350
 	1    0    0    -1
 $EndComp
@@
 L power:+5V #PWR015
 U 1 1 618FEF67
-P 850 1200
-F 0 "#PWR015" H 850 1050 50  0001 C CNN
-F 1 "+5V" H 865 1373 50  0000 C CNN
-F 2 "" H 850 1200 50  0001 C CNN
-F 3 "" H 850 1200 50  0001 C CNN
-	1    850  1200
+P 800 1200
+F 0 "#PWR015" H 800 1050 50  0001 C CNN
+F 1 "+5V" H 815 1373 50  0000 C CNN
+F 2 "" H 800 1200 50  0001 C CNN
+F 3 "" H 800 1200 50  0001 C CNN
+	1    800  1200
 	1    0    0    -1
 $EndComp
@@
 L power:GND #PWR016
 U 1 1 61917F0E
-P 850 1500
-F 0 "#PWR016" H 850 1250 50  0001 C CNN
-F 1 "GND" H 855 1327 50  0000 C CNN
-F 2 "" H 850 1500 50  0001 C CNN
-F 3 "" H 850 1500 50  0001 C CNN
-	1    850  1500
-	1    0    0    -1
-$EndComp
-Wire Wire Line
-	800  1450 850  1450
-Wire Wire Line
-	850  1450 850  1500
-Wire Wire Line
-	800  1250 850  1250
-Wire Wire Line
-	850  1250 850  1200
-Wire Wire Line
-	800  1350 950  1350
+P 800 1500
+F 0 "#PWR016" H 800 1250 50  0001 C CNN
+F 1 "GND" H 805 1327 50  0000 C CNN
+F 2 "" H 800 1500 50  0001 C CNN
+F 3 "" H 800 1500 50  0001 C CNN
+	1    800  1500
+	1    0    0    -1
+$EndComp
+Wire Wire Line
+	750  1450 800  1450
+Wire Wire Line
+	800  1450 800  1500
+Wire Wire Line
+	750  1250 800  1250
+Wire Wire Line
+	800  1250 800  1200
+Wire Wire Line
+	750  1350 900  1350
 $Comp
 L power:PWR_FLAG #FLG02
@@
 Wire Wire Line
 	13600 8300 13600 8450
+$Comp
+L power:+5V #PWR0147
+U 1 1 617975E6
+P 6800 6650
+F 0 "#PWR0147" H 6800 6500 50  0001 C CNN
+F 1 "+5V" H 6815 6823 50  0000 C CNN
+F 2 "" H 6800 6650 50  0001 C CNN
+F 3 "" H 6800 6650 50  0001 C CNN
+	1    6800 6650
+	-1   0    0    -1
+$EndComp
+$Comp
+L power:GND #PWR0148
+U 1 1 617975EC
+P 6800 6950
+F 0 "#PWR0148" H 6800 6700 50  0001 C CNN
+F 1 "GND" H 6805 6777 50  0000 C CNN
+F 2 "" H 6800 6950 50  0001 C CNN
+F 3 "" H 6800 6950 50  0001 C CNN
+	1    6800 6950
+	-1   0    0    -1
+$EndComp
+Wire Wire Line
+	6850 6900 6800 6900
+Wire Wire Line
+	6800 6900 6800 6950
+Wire Wire Line
+	6850 6700 6800 6700
+Wire Wire Line
+	6800 6700 6800 6650
+$Comp
+L Connector:Conn_01x03_Male J2
+U 1 1 617975E0
+P 7050 6800
+F 0 "J2" H 7100 6600 50  0000 C CNN
+F 1 "Conn_01x03_Male" V 7000 6850 50  0000 C CNN
+F 2 "Connector_JST:JST_XH_B3B-XH-A_1x03_P2.50mm_Vertical" H 7050 6800 50  0001 C CNN
+F 3 "~" H 7050 6800 50  0001 C CNN
+	1    7050 6800
+	-1   0    0    -1
+$EndComp
+Wire Wire Line
+	6450 6800 6650 6800
+Text GLabel 3850 8400 0    50   Input ~ 0
+DIN
+Text GLabel 3850 8500 0    50   Input ~ 0
+DOUT
+$Comp
+L Connector:Conn_01x04_Male J3
+U 1 1 61967C1E
+P 4050 8300
+F 0 "J3" H 4022 8274 50  0000 R CNN
+F 1 "Conn_01x04_Male" H 4022 8183 50  0000 R CNN
+F 2 "Connector_PinHeader_2.54mm:PinHeader_1x04_P2.54mm_Vertical" H 4050 8300 50  0001 C CNN
+F 3 "~" H 4050 8300 50  0001 C CNN
+	1    4050 8300
+	-1   0    0    -1
+$EndComp
+$Comp
+L power:GND #PWR?
+U 1 1 6197B305
+P 3850 8300
+F 0 "#PWR?" H 3850 8050 50  0001 C CNN
+F 1 "GND" V 3850 8100 50  0000 C CNN
+F 2 "" H 3850 8300 50  0001 C CNN
+F 3 "" H 3850 8300 50  0001 C CNN
+	1    3850 8300
+	0    1    1    0
+$EndComp
+$Comp
+L power:+5V #PWR?
+U 1 1 6197D265
+P 3850 8200
+F 0 "#PWR?" H 3850 8050 50  0001 C CNN
+F 1 "+5V" V 3850 8400 50  0000 C CNN
+F 2 "" H 3850 8200 50  0001 C CNN
+F 3 "" H 3850 8200 50  0001 C CNN
+	1    3850 8200
+	0    -1   1    0
+$EndComp
+Text GLabel 900  1250 1    50   Input ~ 0
+DIN
+Wire Wire Line
+	900  1350 900  1250
+Wire Wire Line
+	900  1350 950  1350
+Connection ~ 900  1350
+Text GLabel 6650 6550 1    50   Input ~ 0
+DOUT
+Wire Wire Line
+	6650 6550 6650 6800
+Connection ~ 6650 6800
+Wire Wire Line
+	6650 6800 6850 6800
 $EndSCHEMATC
